Commit message: Update sensor.xacro

File: soly/urdf/sensor.xacro (robot description, xacro)
@@ -1,322 +1,61 @@
 <?xml version="1.0"?>
 <robot xmlns:xacro="http://ros.org/wiki/xacro" name="robot">
-<xacro:include filename="$(find soly)/urdf/robot.gazebo" />
- <link
-    name="lidar_link">
+  <link name="lidar_link">
     <inertial>
-      <origin
-        xyz="-0.030032 -1.4396E-05 -0.011702"
-        rpy="0 0 0" />
-      <mass
-        value="0.20673" />
-      <inertia
-        ixx="9.8581E-05"
-        ixy="6.059E-08"
-        ixz="2.731E-06"
-        iyy="9.3988E-05"
-        iyz="3.6075E-08"
-        izz="0.00013743" />
+      <origin xyz="-0.0300318871029288 -1.4396172640152E-05 -0.0117015085354246" rpy="0 0 0" />
+      <mass value="0.206728439544989" />
+      <inertia ixx="9.85814795131668E-05" ixy="6.05897051150735E-08" ixz="2.73099304949762E-06"
+               iyy="9.39878643673402E-05" iyz="3.60751965637769E-08" izz="0.000137433441323384" />
     </inertial>
     <visual>
-      <origin
-        xyz="0 0 0"
-        rpy="0 0 0" />
+      <origin xyz="0 0 0" rpy="0 0 0" />
       <geometry>
-        <mesh
-          filename="package://soly/meshes/lidar_link.STL" />
+        <mesh filename="package://soly/meshes/lidar_link.STL" />
       </geometry>
-      <material
-        name="">
-        <color
-          rgba="0.69804 0.69804 0.69804 1" />
+      <material name="lidar_material">
+        <color rgba="0.698 0.698 0.698 1" />
       </material>
     </visual>
     <collision>
-      <origin
-        xyz="0 0 0"
-        rpy="0 0 0" />
+      <origin xyz="0 0 0" rpy="0 0 0" />
       <geometry>
-        <mesh
-          filename="package://soly/meshes/lidar_link.STL" />
+        <mesh filename="package://soly/meshes/lidar_link.STL" />
       </geometry>
     </collision>
   </link>
-  <joint
-    name="lidar_joint"
-    type="fixed">
-    <origin
-      xyz="0.0382071011949748 -0.00268801927161358 0.0927452794745628"
-      rpy="0 0 0" />
-    <parent
-      link="base_link" />
-    <child
-      link="lidar_link" />
-    <axis
-      xyz="0 0 0" />
+  <joint name="lidar_joint" type="fixed">
+    <origin xyz="0.029596 -0.0037429 0.095257" rpy="0 0 0" />
+    <parent link="base_link" />
+    <child link="lidar_link" />
+    <dontPublish>true</dontPublish> <!-- Add this line -->
   </joint>
-  <link
-    name="ultrasonic_link">
+  <link name="ultrasonic_link">
     <inertial>
-      <origin
-        xyz="-0.0135129398527417 -0.000885994358649722 0.000138154717298"
-        rpy="0 0 0" />
-      <mass
-        value="0.00391542529593063" />
-      <inertia
-        ixx="3.1796509412328E-07"
-        ixy="9.46214068032248E-22"
-        ixz="-3.2817516054534E-11"
-        iyy="1.03578988309517E-07"
-        iyz="1.13097335529236E-09"
-        izz="2.48381258422786E-07" />
+      <origin xyz="-0.0135129398527418 -0.000885994358649805 0.000138154717298" rpy="0 0 0" />
+      <mass value="0.00391542529593063" />
+      <inertia ixx="3.1796509412328E-07" ixy="1.79491252116504E-23" ixz="-3.28175160545291E-11"
+               iyy="1.03578988309517E-07" iyz="1.13097335529237E-09" izz="2.48381258422786E-07" />
     </inertial>
     <visual>
-      <origin
-        xyz="0 0 0"
-        rpy="0 0 0" />
+      <origin xyz="0 0 0" rpy="0 0 0" />
       <geometry>
-        <mesh
-          filename="package://soly/meshes/ultrasonic_link.STL" />
+        <mesh filename="package://soly/meshes/ultrasonic_link.STL" />
       </geometry>
-      <material
-        name="">
-        <color
-          rgba="0.792156862745098 0.819607843137255 0.933333333333333 1" />
+      <material name="ultrasonic_material">
+        <color rgba="0.792 0.820 0.933 1" />
       </material>
     </visual>
     <collision>
-      <origin
-        xyz="0 0 0"
-        rpy="0 0 0" />
+      <origin xyz="0 0 0" rpy="0 0 0" />
       <geometry>
-        <mesh
-          filename="package://soly/meshes/ultrasonic_link.STL" />
+        <mesh filename="package://soly/meshes/ultrasonic_link.STL" />
       </geometry>
     </collision>
   </link>
-  <joint
-    name="ultrasonic_joint"
-    type="fixed">
-    <origin
-      xyz="0.211240668525376 -0.00215148294074055 -0.0186747771202758"
-      rpy="0 0 0" />
-    <parent
-      link="base_link" />
-    <child
-      link="ultrasonic_link" />
-    <axis
-      xyz="0 0 0" />
+  <joint name="ultrasonic_joint" type="fixed">
+    <origin xyz="0.20263 -0.0032064 -0.013163" rpy="0 0 0" />
+    <parent link="base_link" />
+    <child link="ultrasonic_link" />
+   <dontPublish>true</dontPublish> <!-- Add this line -->
   </joint>
- <link
-    name="ir1_link">
-    <inertial>
-      <origin
-        xyz="-0.00481362751522246 0.00132001853896842 0.000172882161482063"
-        rpy="0 0 0" />
-      <mass
-        value="0.00401886169206222" />
-      <inertia
-        ixx="3.93267840144752E-07"
-        ixy="2.98939269827619E-09"
-        ixz="8.86513169312633E-10"
-        iyy="1.06592751976012E-07"
-        iyz="5.62188584345873E-08"
-        izz="3.6011763814111E-07" />
-    </inertial>
-    <visual>
-      <origin
-        xyz="0 0 0"
-        rpy="0 0 0" />
-      <geometry>
-        <mesh
-          filename="package://soly/meshes/ir1_link.STL" />
-      </geometry>
-      <material
-        name="">
-        <color
-          rgba="0.698039215686274 0.698039215686274 0.698039215686274 1" />
-      </material>
-    </visual>
-    <collision>
-      <origin
-        xyz="0 0 0"
-        rpy="0 0 0" />
-      <geometry>
-        <mesh
-          filename="package://soly/meshes/ir1_link.STL" />
-      </geometry>
-    </collision>
-  </link>
-  <joint
-    name="ir1_joint"
-    type="fixed">
-    <origin
-      xyz="0.195955295219554 0.0385044353139036 -0.0532547771202757"
-      rpy="3.14159265358979 1.5707963267949 0" />
-    <parent
-      link="base_link" />
-    <child
-      link="ir1_link" />
-    <axis
-      xyz="0 0 0" />
-  </joint>
-  <link
-    name="ir2_link">
-    <inertial>
-      <origin
-        xyz="-0.00481362801677537 -0.00113558714623704 -0.000694835026359641"
-        rpy="0 0 0" />
-      <mass
-        value="0.00401886327181738" />
-      <inertia
-        ixx="3.93268120546107E-07"
-        ixy="-2.37043296433581E-09"
-        ixz="-2.02579070933095E-09"
-        iyy="1.06755791464812E-07"
-        iyz="-5.65850445734827E-08"
-        izz="3.59954836064108E-07" />
-    </inertial>
-    <visual>
-      <origin
-        xyz="0 0 0"
-        rpy="0 0 0" />
-      <geometry>
-        <mesh
-          filename="package://soly/meshes/ir2_link.STL" />
-      </geometry>
-      <material
-        name="">
-        <color
-          rgba="0.698039215686274 0.698039215686274 0.698039215686274 1" />
-      </material>
-    </visual>
-    <collision>
-      <origin
-        xyz="0 0 0"
-        rpy="0 0 0" />
-      <geometry>
-        <mesh
-          filename="package://soly/meshes/ir2_link.STL" />
-      </geometry>
-    </collision>
-  </link>
-  <joint
-    name="ir2_joint"
-    type="fixed">
-    <origin
-      xyz="0.196524000604301 -0.0412038414361793 -0.0532547771202757"
-      rpy="0 1.5707963267949 0" />
-    <parent
-      link="base_link" />
-    <child
-      link="ir2_link" />
-    <axis
-      xyz="0 0 0" />
-  </joint>
-  <link
-    name="ir3_link">
-    <inertial>
-      <origin
-        xyz="-0.00481362699767693 -0.000356632379966471 -0.00128264314024309"
-        rpy="0 0 0" />
-      <mass
-        value="0.00401885992553366" />
-      <inertia
-        ixx="3.9326752284973E-07"
-        ixy="-3.51976309367688E-10"
-        ixz="-3.09818608179275E-09"
-        iyy="2.80971080995922E-07"
-        iyz="-1.30238099937933E-07"
-        izz="1.85739047870527E-07" />
-    </inertial>
-    <visual>
-      <origin
-        xyz="0 0 0"
-        rpy="0 0 0" />
-      <geometry>
-        <mesh
-          filename="package://soly/meshes/ir3_link.STL" />
-      </geometry>
-      <material
-        name="">
-        <color
-          rgba="0.698039215686274 0.698039215686274 0.698039215686274 1" />
-      </material>
-    </visual>
-    <collision>
-      <origin
-        xyz="0 0 0"
-        rpy="0 0 0" />
-      <geometry>
-        <mesh
-          filename="package://soly/meshes/ir3_link.STL" />
-      </geometry>
-    </collision>
-  </link>
-  <joint
-    name="ir3_joint"
-    type="fixed">
-    <origin
-      xyz="0.119808606366819 -0.15892448730863 -0.0532547771202758"
-      rpy="0 1.5707963267949 0" />
-    <parent
-      link="base_link" />
-    <child
-      link="ir3_link" />
-    <axis
-      xyz="0 0 0" />
-  </joint>
-  <link
-    name="ir4_link">
-    <inertial>
-      <origin
-        xyz="-0.00481362670731214 -0.00108331607509763 0.00077381911838259"
-        rpy="0 0 0" />
-      <mass
-        value="0.0040188584332583" />
-      <inertia
-        ixx="3.93267300685738E-07"
-        ixy="-2.79095960373661E-09"
-        ixz="1.39038933506485E-09"
-        iyy="2.80594324911853E-07"
-        iyz="1.30375094152064E-07"
-        izz="1.8611562393443E-07" />
-    </inertial>
-    <visual>
-      <origin
-        xyz="0 0 0"
-        rpy="0 0 0" />
-      <geometry>
-        <mesh
-          filename="package://soly/meshes/ir4_link.STL" />
-      </geometry>
-      <material
-        name="">
-        <color
-          rgba="0.698039215686274 0.698039215686274 0.698039215686274 1" />
-      </material>
-    </visual>
-    <collision>
-      <origin
-        xyz="0 0 0"
-        rpy="0 0 0" />
-      <geometry>
-        <mesh
-          filename="package://soly/meshes/ir4_link.STL" />
-      </geometry>
-    </collision>
-  </link>
-  <joint
-    name="ir4_joint"
-    type="fixed">
-    <origin
-      xyz="0.117567961905311 0.155118448852247 -0.0532547771202757"
-      rpy="0 1.5707963267949 0" />
-    <parent
-      link="base_link" />
-    <child
-      link="ir4_link" />
-    <axis
-      xyz="0 0 0" />
-  </joint>
-  </robot>
+</robot>
